Commit message: Update robot_description links to match the SKD-1 sensors

File: skd1_description/urdf/skd1_core.urdf.xacro (robot description, xacro)
@@ -82,15 +82,15 @@
 	</xacro:skd1_wheel>
     <!-- Sensors -->
-	<!-- MTI630 IMU -->
-	<link name="xsens_imu_link">
+	<!-- Phidgets Spatial IMU -->
+	<link name="phidgets_imu_link">
 		<xacro:dummy_inertial />
 	</link>
-	<joint name="xsens_imu_joint" type="fixed">
+	<joint name="phidgets_imu_joint" type="fixed">
 		<parent link="base_link" />
-		<child link="xsens_imu_link" />
+		<child link="phidgets_imu_link" />
 		<origin xyz="0 0 0.05" rpy="0 0 0" />
 	</joint>
 	<!-- RPLidar S3 -->
-	<link name="rplidar_s3_link">
+	<link name="rplidar_link">
 		<xacro:dummy_inertial />
 		<collision>
@@ -109,5 +109,5 @@
 	<joint name="rplidar_joint" type="fixed">
 		<parent link="base_link"/>
-		<child link="rplidar_s3_link"/>
+		<child link="rplidar_link"/>
 		<origin xyz="0.0 0.0 ${chassis_z_size/2 + 0.16}" rpy="0 0 ${pi}"/>
 	</joint>

File: skd1_description/urdf/skd1_sim_sensors.urdf.xacro (robot description, xacro)
@@ -1,19 +1,19 @@
 <?xml version="1.0"?>
 <robot xmlns:xacro="http://www.ros.org/wiki/xacro">
-<gazebo reference="xsens_imu_link">
-    <sensor name="xsens_imu" type="imu">
+<gazebo reference="phidgets_imu_link">
+    <sensor name="phidgets_imu" type="imu">
         <always_on>1</always_on>
         <update_rate>20</update_rate>
         <visualize>true</visualize>
-        <topic>mti_630_8A1G6/imu/data</topic>
-        <gz_frame_id>xsens_imu_link</gz_frame_id>
+        <topic>phidgets_373223/imu/data</topic>
+        <gz_frame_id>phidgets_imu_link</gz_frame_id>
         <!-- <enable_metrics>true</enable_metrics> -->
     </sensor>
-    <sensor name="xsens_mag" type="magnetometer">
+    <sensor name="phidgets_mag" type="magnetometer">
         <always_on>1</always_on>
         <update_rate>20</update_rate>
         <visualize>true</visualize>
-        <topic>mti_630_8A1G6/imu/mag</topic>
-        <gz_frame_id>xsens_imu_link</gz_frame_id>
+        <topic>phidgets_373223/imu/mag</topic>
+        <gz_frame_id>phidgets_imu_link</gz_frame_id>
         <!-- <enable_metrics>true</enable_metrics> -->
     </sensor>

Commit message: Update diff_drive_controller and URDF to match SKD1 dimensions.

File: skd1_description/urdf/skd1_core.urdf.xacro (robot description, xacro)
@@ -4,7 +4,7 @@
     <xacro:include filename="$(find skd1_description)/urdf/wheel.urdf.xacro" />
 	<!--  Wheel distance between front and rear -->
-	<xacro:property name="wheel_distance" value="0.25" />
+	<xacro:property name="wheel_distance" value="0.20" />
 	<!-- Wheel distance between left and right side -->
-	<xacro:property name="wheel_separation" value="0.475" />
+	<xacro:property name="wheel_separation" value="0.33" />
 	<!-- Wheel properties -->
 	<xacro:property name="wheel_mass" value="0.150" />
@@ -12,13 +12,14 @@
 	<xacro:property name="wheel_width" value="0.06" />
 	<!-- Chassis size -->
-	<xacro:property name="chassis_x_size" value="0.45" />
-	<xacro:property name="chassis_y_size" value="0.38" />
-	<xacro:property name="chassis_z_size" value="0.05" />
+	<xacro:property name="chassis_x_size" value="0.40" />
+	<xacro:property name="chassis_y_size" value="0.25" />
+	<xacro:property name="chassis_z_size" value="0.09" />
 	<!-- https://docs.ros.org/en/humble/Tutorials/Intermediate/URDF/Adding-Physical-and-Collision-Properties-to-a-URDF-Model.html -->
     <link name="base_link">
 		<visual>
-    		<origin xyz="0 0 0" rpy="0 0 0" />
+    		<origin xyz="0 0 0" rpy="${(pi/2)} 0 ${-(pi/2)}" />
 			<geometry>
-				<box size="${chassis_x_size} ${chassis_y_size} ${chassis_z_size}"/>
+				<mesh filename="file://$(find skd1_description)/meshes/skd1_chassis.stl" scale="0.001 0.001 0.001" />
+				<!-- <box size="${chassis_x_size} ${chassis_y_size} ${chassis_z_size}"/> -->
 			</geometry>
 			<material name="Red">
@@ -32,5 +33,5 @@
 			</geometry>
 		</collision>
-		<visual>
+		<!-- <visual>
     		<origin xyz="${chassis_x_size/2 + 0.045} 0 ${chassis_z_size/2 + 0.06}" rpy="0 0 0" />
 			<geometry>
@@ -46,5 +47,5 @@
 				<box size="0.09 0.17 0.12"/>
 			</geometry>
-		</collision>
+		</collision>-->
     </link>
 	<!-- Base footprint is on the ground under the robot -->

Commit message: Update meshes and URDF dimensions and positions

File: skd1_description/urdf/skd1_core.urdf.xacro (robot description, xacro)
@@ -3,8 +3,10 @@
     <xacro:include filename="$(find skd1_description)/urdf/inertial_macros.xacro" />
     <xacro:include filename="$(find skd1_description)/urdf/wheel.urdf.xacro" />
-	<!--  Wheel distance between front and rear -->
-	<xacro:property name="wheel_distance" value="0.20" />
-	<!-- Wheel distance between left and right side -->
-	<xacro:property name="wheel_separation" value="0.33" />
+	<!-- Distance between front and rear wheel axles (wheelbase) -->
+	<xacro:property name="wheel_distance" value="0.21524" />
+	<!-- Distance between the centerlines of the left and right wheels (track width) -->
+	<xacro:property name="wheel_separation" value="0.37068" />
+	<!-- Z-coordinate of the wheel axle relative to base_link -->
+	<xacro:property name="wheel_height" value="0.0328" />
 	<!-- Wheel properties -->
 	<xacro:property name="wheel_mass" value="0.150" />
@@ -12,40 +14,66 @@
 	<xacro:property name="wheel_width" value="0.06" />
 	<!-- Chassis size -->
-	<xacro:property name="chassis_x_size" value="0.40" />
-	<xacro:property name="chassis_y_size" value="0.25" />
-	<xacro:property name="chassis_z_size" value="0.09" />
-	<!-- https://docs.ros.org/en/humble/Tutorials/Intermediate/URDF/Adding-Physical-and-Collision-Properties-to-a-URDF-Model.html -->
-    <link name="base_link">
+	<xacro:property name="chassis_x_size" value="0.410" />
+	<xacro:property name="chassis_y_size" value="0.260" />
+	<xacro:property name="chassis_z_size" value="0.094" />
+	<!-- The 'base_link' is located at the geometric center of the chassis
+     (center of the acrylic plate) and positioned above it (5 mm thickness) -->
+	<link name="base_link">
 		<visual>
-    		<origin xyz="0 0 0" rpy="${(pi/2)} 0 ${-(pi/2)}" />
+    		<origin xyz="0 0 0" rpy="${(pi/2)} 0 ${pi}"/>
 			<geometry>
 				<mesh filename="file://$(find skd1_description)/meshes/skd1_chassis.stl" scale="0.001 0.001 0.001" />
 				<!-- <box size="${chassis_x_size} ${chassis_y_size} ${chassis_z_size}"/> -->
 			</geometry>
-			<material name="Red">
-				<color rgba="${255/255} ${0/255} ${0/255} 1.0"/>
+			<material name="White">
+				<color rgba="1.0 1.0 1.0 1.0"/>
 			</material>
 		</visual>
+		<xacro:property name="chassis_z_offset" value="0.005" />
+		<!-- Chassis -->
 		<collision>
-			<origin xyz="0 0 0"/>
+			<origin xyz="0 0 ${chassis_z_size/2-chassis_z_offset}"/>
 			<geometry>
 				<box size="${chassis_x_size} ${chassis_y_size} ${chassis_z_size}"/>
 			</geometry>
 		</collision>
-		<!-- <visual>
-    		<origin xyz="${chassis_x_size/2 + 0.045} 0 ${chassis_z_size/2 + 0.06}" rpy="0 0 0" />
+		<!-- Antenna deck -->
+		<xacro:property name="deck_x_size" value="0.150" />
+		<xacro:property name="deck_y_size" value="0.260" />
+		<xacro:property name="deck_z_size" value="0.187" />
+		<collision>
+			<origin xyz="0 0 ${deck_z_size/2+0.089}"/>
 			<geometry>
-				<box size="0.09 0.17 0.12"/>
+				<box size="${deck_x_size} ${deck_y_size} ${deck_z_size}"/>
 			</geometry>
-			<material name="Green">
-				<color rgba="${0/255} ${255/255} ${0/255} 1.0"/>
-			</material>
-		</visual>
-		<collision>
-			<origin xyz="${chassis_x_size/2 + 0.045} 0 ${chassis_z_size/2 + 0.06}" rpy="0 0 0" />
+		</collision>
+		<!-- Motor covers -->
+		<xacro:property name="mcover_x_size" value="0.0976" />
+		<xacro:property name="mcover_y_size" value="0.083" />
+		<xacro:property name="mcover_z_size" value="0.0476" />
+		<collision> <!-- Front Left-->
+			<origin xyz="${wheel_distance/2} ${chassis_y_size/2-mcover_y_size/2} ${-mcover_z_size/2-chassis_z_offset}"/>
 			<geometry>
-				<box size="0.09 0.17 0.12"/>
+				<box size="${mcover_x_size} ${mcover_y_size} ${mcover_z_size}"/>
 			</geometry>
-		</collision>-->
+		</collision>
+		<collision> <!-- Front Right-->
+			<origin xyz="${wheel_distance/2} -${chassis_y_size/2-mcover_y_size/2} ${-mcover_z_size/2-chassis_z_offset}"/>
+			<geometry>
+				<box size="${mcover_x_size} ${mcover_y_size} ${mcover_z_size}"/>
+			</geometry>
+		</collision>
+		<collision> <!-- Rear Left-->
+			<origin xyz="-${wheel_distance/2} ${chassis_y_size/2-mcover_y_size/2} ${-mcover_z_size/2-chassis_z_offset}"/>
+			<geometry>
+				<box size="${mcover_x_size} ${mcover_y_size} ${mcover_z_size}"/>
+			</geometry>
+		</collision>
+		<collision> <!-- Rear Right-->
+			<origin xyz="-${wheel_distance/2} -${chassis_y_size/2-mcover_y_size/2} ${-mcover_z_size/2-chassis_z_offset}"/>
+			<geometry>
+				<box size="${mcover_x_size} ${mcover_y_size} ${mcover_z_size}"/>
+			</geometry>
+		</collision>
     </link>
 	<!-- Base footprint is on the ground under the robot -->
@@ -54,5 +82,5 @@
 	</link>
     <joint name="base_footprint_joint" type="fixed">
-        <origin xyz="0 0 ${-wheel_radius}" rpy="0 0 0" />
+        <origin xyz="0 0 -${wheel_height+wheel_radius}" rpy="0 0 0" />
         <parent link="base_link" />
         <child link="base_footprint" />
@@ -60,5 +88,5 @@
 	<!-- Interial link stores the robot's inertial information -->
     <link name="inertial_link">
-		<xacro:inertial_box mass="2.0" x="${chassis_x_size}" y="${chassis_y_size}" z="${chassis_z_size}">
+		<xacro:inertial_box mass="5.0" x="${chassis_x_size}" y="${chassis_y_size}" z="${chassis_z_size}">
             <origin xyz="0 0 0" rpy="0 0 0"/>
         </xacro:inertial_box>
@@ -71,18 +99,26 @@
 	<!-- Wheel macros -->
 	<xacro:skd1_wheel wheel_prefix="front_left">
-		<origin xyz="${wheel_distance/2} ${wheel_separation/2} 0" rpy="0 0 0" />
+		<origin xyz="${wheel_distance/2} ${wheel_separation/2} -${wheel_height}" rpy="0 0 0" />
 	</xacro:skd1_wheel>
 	<xacro:skd1_wheel wheel_prefix="front_right">
-		<origin xyz="${wheel_distance/2} ${-wheel_separation/2} 0" rpy="0 0 0" />
+		<origin xyz="${wheel_distance/2} ${-wheel_separation/2} -${wheel_height}" rpy="0 0 0" />
 	</xacro:skd1_wheel>
 	<xacro:skd1_wheel wheel_prefix="rear_left">
-		<origin xyz="${-wheel_distance/2} ${wheel_separation/2} 0" rpy="0 0 0" />
+		<origin xyz="${-wheel_distance/2} ${wheel_separation/2} -${wheel_height}" rpy="0 0 0" />
 	</xacro:skd1_wheel>
 	<xacro:skd1_wheel wheel_prefix="rear_right">
-		<origin xyz="${-wheel_distance/2} ${-wheel_separation/2} 0" rpy="0 0 0" />
+		<origin xyz="${-wheel_distance/2} ${-wheel_separation/2} -${wheel_height}" rpy="0 0 0" />
 	</xacro:skd1_wheel>
     <!-- Sensors -->
 	<!-- Phidgets Spatial IMU -->
 	<link name="phidgets_imu_link">
+		<visual>
+			<geometry>
+				<box size="0.037846 0.038989 0.01338"/>
+			</geometry>
+			<material name="Magenta">
+				<color rgba="1.0 0.0 1.0 1.0"/>
+			</material>
+		</visual>
 		<xacro:dummy_inertial />
 	</link>
@@ -90,28 +126,40 @@
 		<parent link="base_link" />
 		<child link="phidgets_imu_link" />
-		<origin xyz="0 0 0.05" rpy="0 0 0" />
+		<origin xyz="0 0 ${0.085-0.006-0.00581}" rpy="0 0 0" />
 	</joint>
-	<!-- RPLidar S3 -->
+	<!-- RPLidar C1 -->
 	<link name="rplidar_link">
-		<xacro:dummy_inertial />
+		<visual>
+			<origin xyz="0 0 -0.0298" rpy="0 0 0"/>
+			<geometry>
+				<mesh filename="file://$(find skd1_description)/meshes/RPLidar_C1M1.stl"  scale="0.001 0.001 0.001"/>
+			</geometry>
+			<material name="Cyan">
+				<color rgba="0.0 1.0 1.0 1.0"/>
+			</material>
+		</visual>
 		<collision>
-			<origin xyz="0 0 0" rpy="0 0 0"/>
+			<origin xyz="0 0 ${-0.0298+0.042/2}" rpy="0 0 0"/>
 			<geometry>
-				<box size="0.06 0.056 0.042"/>
+				<box size="0.056 0.056 0.042"/>
 			</geometry>
 		</collision>
-		<visual>
-			<origin xyz="0 0 0" rpy="${pi/2} 0 ${-pi/2}"/>
-			<geometry>
-				<mesh filename="file://$(find skd1_description)/meshes/rplidar_s3.stl"  scale="0.001 0.001 0.001"/>
-			</geometry>
-		</visual>
+		<xacro:dummy_inertial />
 	</link>
 	<joint name="rplidar_joint" type="fixed">
 		<parent link="base_link"/>
 		<child link="rplidar_link"/>
-		<origin xyz="0.0 0.0 ${chassis_z_size/2 + 0.16}" rpy="0 0 ${pi}"/>
+		<origin xyz="0.075 0 ${chassis_z_size-0.005+0.005+0.0298}" rpy="0 0 0"/>
 	</joint>
 	<link name="ardusimple_gps_link">
+		<visual>
+			<origin xyz="0 0 0" rpy="0 0 ${pi/2}"/>
+			<geometry>
+				<mesh filename="file://$(find skd1_description)/meshes/uBlox_ANT2B-ANN.stl"  scale="0.001 0.001 0.001"/>
+			</geometry>
+			<material name="Yellow">
+				<color rgba="1.0 1.0 0.0 1.0"/>
+			</material>
+		</visual>
 		<xacro:dummy_inertial />
 	</link>
@@ -119,5 +167,5 @@
 		<parent link="base_link" />
 		<child link="ardusimple_gps_link" />
-		<origin xyz="0.0 -0.1 0.2" rpy="0 0 0" />
+		<origin xyz="0 0.055 0.282" rpy="0 0 0" />
 	</joint>
 	<link name="m8n_gps_link">
@@ -127,5 +175,5 @@
 		<parent link="base_link" />
 		<child link="m8n_gps_link" />
-		<origin xyz="0.0 0.1 0.2" rpy="0 0 0" />
+		<origin xyz="0 -0.055 0.282" rpy="0 0 0" />
 	</joint>
 </robot>

File: skd1_description/urdf/wheel.urdf.xacro (robot description, xacro)
@@ -23,10 +23,13 @@
                     </xacro:if>
                 </geometry>
+                <material name="Dark gray">
+                    <color rgba="0.175 0.175 0.175 1.0"/>
+                </material>
             </visual>
             <collision>
                 <origin xyz="0 0 0" rpy="${pi/2} 0 0"/>
                 <geometry>
-                    <!-- <cylinder radius="${wheel_radius}" length="${wheel_width}"/> -->
-                    <sphere radius="${wheel_radius}"/>
+                    <cylinder radius="${wheel_radius}" length="${wheel_width}"/>
+                    <!-- <sphere radius="${wheel_radius}"/> -->
                 </geometry>
             </collision>

Commit message: Update URDF to match RPLIDAR C1 measurements orientation.

File: skd1_description/urdf/skd1_core.urdf.xacro (robot description, xacro)
@@ -150,5 +150,5 @@
 		<parent link="base_link"/>
 		<child link="rplidar_link"/>
-		<origin xyz="0.075 0 ${chassis_z_size-0.005+0.005+0.0298}" rpy="0 0 0"/>
+		<origin xyz="0.075 0 ${chassis_z_size-0.005+0.005+0.0298}" rpy="0 0 ${pi}"/>
 	</joint>
 	<link name="ardusimple_gps_link">
